File: MainBoard/MainBoard.kicad_sch (KiCad schematic)
At the start: 41 parts, among them U1 TL074CN, U2 TL074CN, U3 TL074CN

Commit message: updated placement
Parts:
- D1: value 1N5934B -> 1N5394B; footprint 1N5934B:P2_DO-201 -> 1N5349B:P2_DO-201
- D2: value 1N5934B -> 1N5349B; footprint 1N5934B:P2_DO-201 -> 1N5349B:P2_DO-201
Connections:
- net Output10: now also Jheader2.8; no longer Jheader2.14
- net Output5: now also Jheader2.12; no longer Jheader2.7
- net Output6: now also Jheader2.14; no longer Jheader2.8
- net Output8: now also Jheader2.13; no longer Jheader2.12
- net Output9: now also Jheader2.7; no longer Jheader2.13
Changed lines of the file:
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@@
     )
   )
-  (global_label "Output8" (shape input) (at 205.74 114.3 180) (fields_autoplaced)
-    (effects (font (size 1.27 1.27)) (justify right))
-    (property "Intersheetrefs" "${INTERSHEET_REFS}" (at 195.8883 114.2206 0)
+  (global_label "Output8" (shape input) (at 205.74 118.11 180) (fields_autoplaced)
+    (effects (font (size 1.27 1.27)) (justify right))
+    (property "Intersheetrefs" "${INTERSHEET_REFS}" (at 195.8883 118.0306 0)
       (effects (font (size 1.27 1.27)) (justify right) hide)
     )
@@
     )
   )
-  (global_label "Output10" (shape input) (at 205.74 121.92 180) (fields_autoplaced)
-    (effects (font (size 1.27 1.27)) (justify right))
-    (property "Intersheetrefs" "${INTERSHEET_REFS}" (at 194.6788 121.9994 0)
+  (global_label "Output10" (shape input) (at 205.74 99.06 180) (fields_autoplaced)
+    (effects (font (size 1.27 1.27)) (justify right))
+    (property "Intersheetrefs" "${INTERSHEET_REFS}" (at 194.6788 99.1394 0)
       (effects (font (size 1.27 1.27)) (justify right) hide)
     )
@@
     )
   )
-  (global_label "Output9" (shape input) (at 205.74 118.11 180) (fields_autoplaced)
-    (effects (font (size 1.27 1.27)) (justify right))
-    (property "Intersheetrefs" "${INTERSHEET_REFS}" (at 195.8883 118.1894 0)
+  (global_label "Output9" (shape input) (at 205.74 95.25 180) (fields_autoplaced)
+    (effects (font (size 1.27 1.27)) (justify right))
+    (property "Intersheetrefs" "${INTERSHEET_REFS}" (at 195.8883 95.3294 0)
       (effects (font (size 1.27 1.27)) (justify right) hide)
     )
@@
     )
   )
-  (global_label "Output6" (shape input) (at 205.74 99.06 180) (fields_autoplaced)
-    (effects (font (size 1.27 1.27)) (justify right))
-    (property "Intersheetrefs" "${INTERSHEET_REFS}" (at 195.8883 98.9806 0)
+  (global_label "Output6" (shape input) (at 205.74 121.92 180) (fields_autoplaced)
+    (effects (font (size 1.27 1.27)) (justify right))
+    (property "Intersheetrefs" "${INTERSHEET_REFS}" (at 195.8883 121.8406 0)
       (effects (font (size 1.27 1.27)) (justify right) hide)
     )
@@
     )
   )
-  (global_label "Output5" (shape input) (at 205.74 95.25 180) (fields_autoplaced)
-    (effects (font (size 1.27 1.27)) (justify right))
-    (property "Intersheetrefs" "${INTERSHEET_REFS}" (at 195.8883 95.1706 0)
+  (global_label "Output5" (shape input) (at 205.74 114.3 180) (fields_autoplaced)
+    (effects (font (size 1.27 1.27)) (justify right))
+    (property "Intersheetrefs" "${INTERSHEET_REFS}" (at 195.8883 114.2206 0)
       (effects (font (size 1.27 1.27)) (justify right) hide)
     )
@@
       (effects (font (size 1.27 1.27)) (justify left))
     )
-    (property "Value" "1N5934B" (at 125.73 155.8924 90)
-      (effects (font (size 1.27 1.27)) (justify left))
-    )
-    (property "Footprint" "1N5934B:P2_DO-201" (at 118.745 154.94 0)
+    (property "Value" "1N5394B" (at 125.73 155.8924 90)
+      (effects (font (size 1.27 1.27)) (justify left))
+    )
+    (property "Footprint" "1N5349B:P2_DO-201" (at 118.745 154.94 0)
       (effects (font (size 1.27 1.27)) hide)
     )
@@
       (effects (font (size 1.27 1.27)) hide)
     )
-    (property "Sim.Library" "../models/TL074.mod" (at 214.63 38.1 0)
+    (property "Sim.Library" "" (at 214.63 38.1 0)
       (effects (font (size 1.27 1.27)) hide)
     )
@@
       (effects (font (size 1.27 1.27)) (justify right))
     )
-    (property "Value" "1N5934B" (at 125.73 168.5924 90)
+    (property "Value" "1N5349B" (at 125.73 168.5924 90)
       (effects (font (size 1.27 1.27)) (justify right))
     )
-    (property "Footprint" "1N5934B:P2_DO-201" (at 127.635 167.64 0)
-      (effects (font (size 1.27 1.27)) hide)
-    )
+    (property "Footprint" "1N5349B:P2_DO-201" (at 127.635 167.64 0)
+      (effects (font (size 1.27 1.27)) hide)
+    )

Commit message: first pass at routing mainboard
Parts:
- added R25: 100k, Resistor_THT:R_Axial_DIN0207_L6.3mm_D2.5mm_P10.16mm_Horizontal, symbol Device:R
- Jheader2: footprint 61301611021:61301611021 -> AMPHENOL_75168-116-20LF; symbol 61301611021:61301611021 -> 75168-116-20LF:75168-116-20LF; MANUFACTURER Samtec -> Amphenol ICC (FCI); PARTREV R -> AL
Connections:
- net GND: now also Jheader2.07, Jheader2.08, Jheader2.09, Jheader2.18
- net InputBus1: now also Jheader2.20; no longer Jheader2.1
- net InputBus2: now also Jheader2.03; no longer Jheader2.2
- net InputBus3: now also Jheader2.06; no longer Jheader2.9
- net InputBus4: now also Jheader2.11; no longer Jheader2.10
- net Output1: now also Jheader2.19; no longer Jheader2.3
- net Output10: now also Jheader2.10; no longer Jheader2.8
- net Output11: now also Jheader2.16; no longer Jheader2.15
- net Output12: now also Jheader2.14; no longer Jheader2.16
- net Output2: now also Jheader2.17; no longer Jheader2.4
- net Output3: now also Jheader2.15; no longer Jheader2.5
- net Output4: now also Jheader2.12; no longer Jheader2.6
- net Output5: now also Jheader2.04; no longer Jheader2.12
- net Output6: now also Jheader2.05; no longer Jheader2.14
- net Output7: now also Jheader2.01; no longer Jheader2.11
- net Output8: now also Jheader2.02; no longer Jheader2.13
- net Output9: now also Jheader2.13; no longer Jheader2.7
- net at U1.12 (4IN+): now also R25.1
